Commit message: Fix IMU sensor. reduced sensor rays

File: description/distance_sensor.xacro (robot description, xacro)
@@ -39,5 +39,5 @@
           <scan>
             <horizontal>
-              <samples>5</samples> <!-- Single ray, 1D distance sensor -->
+              <samples>3</samples> <!-- Single ray, 1D distance sensor -->
               <resolution>1</resolution>
               <min_angle> -0.01 </min_angle>

File: description/imu.xacro (robot description, xacro)
@@ -1,5 +1,5 @@
 <?xml version="1.0"?>
 <robot xmlns:xacro="http://www.ros.org/wiki/xacro">
-    <joint name="imu" type="fixed">
+    <joint name="imu_joint" type="fixed">
         <parent link="chassis"/>
         <child link="imu_link"/>
@@ -13,16 +13,22 @@
             <material name="black"/>
         </visual>
+        <inertial>
+            <mass value="0.001"/>
+            <origin xyz="0.0 0.0 0.0"/>
+            <inertia ixx="0.000001" ixy="0.0" ixz="0.0" iyy="0.000001" iyz="0.0" izz="0.000001"/>
+        </inertial>
     </link>
     <gazebo reference="imu_link">
-        <gravity>false</gravity>
+        <gravity>true</gravity>
     <sensor name="imu_sensor" type="imu">
+        <pose>0 0 0 0 0 0</pose>
         <always_on>true</always_on>
-        <update_rate>10</update_rate>
+        <topic>/imu</topic>
+        <update_rate>10.0</update_rate>
         <visualize>true</visualize>
-        <topic>/imu/data</topic>
         <plugin filename="libgazebo_ros_imu_sensor.so" name="imu_plugin">
-            <topicName>imu</topicName>
+            <topicName>/imu</topicName>
             <bodyName>imu_link</bodyName>
-            <updateRateHZ>10.0</updateRateHZ>
+            <updateRateHZ>100.0</updateRateHZ>
             <gaussianNoise>0.0</gaussianNoise>
             <xyzOffset>0 0 0</xyzOffset>
@@ -30,10 +36,5 @@
             <frameName>imu_link</frameName>
             <initialOrientationAsReference>false</initialOrientationAsReference>
-            <ros>
-                <remapping>/imu_plugin/out:=/imu/data</remapping> <!-- Topic remapping -->
-                <namespace>/simulation</namespace>
-            </ros>
         </plugin>
-        <pose>0 0 0 0 0 0</pose>
     </sensor>
     </gazebo>

File: description/robot.urdf.xacro (robot description, xacro)
@@ -7,5 +7,5 @@
     <!-- <xacro:include filename="gazebo_control.xacro"/> -->
     <xacro:include filename="camera.xacro"/>
-    <!-- <xacro:include filename="imu.xacro"/> -->
+    <xacro:include filename="imu.xacro"/>
     <xacro:distance_sensor prefix="front">
         <origin xyz="0.09 0.0 0.005"/>
